File: PCB/House/House.kicad_pcb (KiCad board)
At the start: 2 copper layers, 95 x 60.5 mm, 37 parts, among them J1 Conn_01x05, U1 HT16K33-28SOP

Commit message: [update] Houseの配線改善(目、ビア位置、屋根裏調整)
* 窓際の表面縦配線の位置を1個内側に移動して目に見えるように修正。
* 各種ビア位置をほぼ線対称になるように移動。
* 屋根裏の裏面配線を外形線に沿うように大きくした。
Routing:
- net Net-(D1-Pad1): track 313.1 -> 357.3 mm
- net GND: track 87.3 -> 120.7 mm, vias 44 -> 34
- net Net-(D19-Pad2): track 98.7 -> 76.1 mm
- net Net-(D17-Pad1): track 197.7 -> 201.4 mm
- net Net-(D18-Pad2): track 123.5 -> 119.8 mm
- net Net-(D23-Pad2): track 84.8 -> 86.6 mm
- net Net-(D22-Pad2): track 73.1 -> 74.7 mm
- net Net-(D21-Pad2): track 62.9 -> 64.0 mm
- net Net-(D1-Pad2): track 82.4 -> 83.3 mm
- net Net-(D25-Pad2): track 108.2 -> 108.4 mm, vias 4 -> 5
- net Net-(D10-Pad2): track 77.9 -> 77.7 mm, vias 4 -> 5
Other:
- board text added: "@ext_sui 2020.02"
- board text removed: "@ext_sui 2020.01"

Commit message: [update] House v1.0登録
* 「シルクからパッドを除外」にチェックを追加(seeed準拠)
* 製造年月を2020.02から2020.03に修正
Other:
- board text added: "@ext_sui 2020.03"
- board text removed: "@ext_sui 2020.02"
Changed lines of the file:
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@@
       (plotvalue true)
       (plotinvisibletext false)
-      (padsonsilk true)
+      (padsonsilk false)
       (subtractmaskfromsilk false)
       (outputformat 1)
@@
     (effects (font (size 1 1) (thickness 0.15)) (justify mirror))
   )
-  (gr_text "@ext_sui 2020.02" (at 169.5 91.5) (layer B.SilkS)
+  (gr_text "@ext_sui 2020.03" (at 169.5 91.5) (layer B.SilkS)
     (effects (font (size 1 1) (thickness 0.2) italic) (justify mirror))
   )
@@
   (gr_line (start 155 100) (end 155 109.5) (layer Edge.Cuts) (width 0.15))
   (gr_line (start 141 110.5) (end 154 110.5) (layer Edge.Cuts) (width 0.15))
-  (segment (start 148.5 97) (end 150.5 97) (width 0.25) (layer B.Cu) (net 2))
-  (via (at 187 65) (size 0.8) (drill 0.4) (layers F.Cu B.Cu) (net 2))
-  (via (at 187 68) (size 0.8) (drill 0.4) (layers F.Cu B.Cu) (net 2))
   (segment (start 142.5 105.92) (end 142.42 106) (width 0.5) (layer B.Cu) (net 1))
   (segment (start 142.5 100.5) (end 142.5 105.92) (width 0.5) (layer B.Cu) (net 1))
@@
   (segment (start 139.75 99) (end 141.75 99) (width 0.5) (layer B.Cu) (net 1))
   (segment (start 142.5 99.75) (end 142.5 100.5) (width 0.5) (layer B.Cu) (net 1))
+  (segment (start 148.5 97) (end 150.5 97) (width 0.25) (layer B.Cu) (net 2))
+  (via (at 187 65) (size 0.8) (drill 0.4) (layers F.Cu B.Cu) (net 2))
+  (via (at 187 68) (size 0.8) (drill 0.4) (layers F.Cu B.Cu) (net 2))
   (via (at 173.5 88.5) (size 0.8) (drill 0.4) (layers F.Cu B.Cu) (net 2))
   (via (at 121.5 88.5) (size 0.8) (drill 0.4) (layers F.Cu B.Cu) (net 2))
