File: PCB/Pillar/Pillar.kicad_pcb (KiCad board)
At the start: 2 copper layers, 100 x 86.6 mm, 29 parts, among them CN1 GROVE_IIC_5V, CN2 GROVE_IIC_5V, CN3 USB_A, CN4 AudioJack3_SwitchTR, CN5 Micro_SD_Card_Det_Hirose_DM3AT, J1 Speaker, SW1 MDOE, SW2 NEXT/VOL+, SW3 PREV/VOL-, U1 SeeeduinoXIAO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

Commit message: (Pcb) 配線改善：ティアドロップ付与と全体の均一 GND ビア打ち #60
Routing:
- net 5V: track 111.0 -> 110.0 mm
- net 3V3: track 186.5 -> 185.6 mm
- net GND: vias 190 -> 283
